Commit message: Update: gripper control working with moveit

File: manipulation/tb4_openmanipulator_moveit/config/turtlebot4.ros2_control.xacro (robot description, xacro)
@@ -43,4 +43,11 @@
                 <state_interface name="velocity"/>
             </joint>
+            <joint name="gripper_right_joint">
+                <command_interface name="position"/>
+                <state_interface name="position">
+                  <param name="initial_value">${initial_positions['gripper_right_joint']}</param>
+                </state_interface>
+                <state_interface name="velocity"/>
+            </joint>
             <joint name="virtual_joint">
                 <command_interface name="position"/>
